File: layouts/example/example.kicad_pcb (KiCad board)
At the start: 2 copper layers, 29 parts

Commit message: Enhance smart placer with simulated annealing and pre-routing validation
Smart Placer improvements:
- Add simulated annealing refinement (now default) for better wire length optimization
- Add force-directed refinement with improvement safeguard
- Add silkscreen text repositioning to avoid component overlaps
- Significant wire length reductions (e.g., power_filter: 113mm -> 46mm)

Autorouter improvements:
- Add PreRoutingValidator class for pre-flight checks
- Validate unconnected pads, overlapping footprints, unplaced components
- Use pad-based bounds for accurate overlap detection
- Block routing on validation errors with actionable messages

Research:
- Add comprehensive autorouting/autoplacement findings document
- Cover Freerouting Python client, OrthoRoute, DeepPCB, KiCad 9 IPC API
- Document force-directed and simulated annealing algorithms

Cleanup:
- Update .gitignore for DSN/SES files, build artifacts, tools
- Remove stale timestamped build files
- Add parts footprints and symbols

All 10 modules placed and routed successfully.

Co-Authored-By: Claude Opus 4.5 <noreply@anthropic.com>
Routing:
- net INT1: track 0.00 -> 71.4 mm, vias 0 -> 2
- net gnd: track 0.00 -> 17.8 mm
- net swdio: track 0.00 -> 6.31 mm, vias 0 -> 1
- net nrst: track 0.00 -> 4.87 mm, vias 0 -> 1
- net vcc_mcu: track 0.00 -> 3.95 mm
